File: PCB/PCB.kicad_sch (KiCad schematic)
At the start: 17 parts, among them U1 ESP32-WROOM-32E-N8R2

Commit message: updates
Parts:
- removed R10, R11, R12, R13, R14, R15, R16, R9: R, Resistor_THT:R_Axial_DIN0207_L6.3mm_D2.5mm_P10.16mm_Horizontal, symbol Device:R
- added J1, J2, J3, J4, J5, J6, J7, J8: Conn_01x02_Pin, symbols_footprint:PinHeader_1x02_P2.54mm_Vertical smd custom, symbol Connector:Conn_01x02_Pin
- added J10: Conn_01x02_Pin, Connector_PinHeader_2.54mm:PinHeader_1x02_P2.54mm_Horizontal, symbol Connector:Conn_01x02_Pin
- added J9: Conn_01x04_Pin, Connector_PinHeader_2.54mm:PinHeader_1x04_P2.54mm_Vertical, symbol Connector:Conn_01x04_Pin
Connections:
- net 3V3: now also J9.1 (Pin_1)
- net GND: now also J1.1 (Pin_1), J10.2 (Pin_2), J2.1 (Pin_1), J3.1 (Pin_1), J4.1 (Pin_1), J5.1 (Pin_1), J6.1 (Pin_1), J7.1 (Pin_1), J8.1 (Pin_1), J9.2 (Pin_2)
- net IO13: now also J1.2 (Pin_2)
- net IO14: now also J2.2 (Pin_2)
- net IO25: now also J5.2 (Pin_2)
- net IO26: now also J4.2 (Pin_2)
- net IO27: now also J3.2 (Pin_2)
- net IO32: now also J7.2 (Pin_2)
- net IO33: now also J6.2 (Pin_2)
- net IO35: now also J8.2 (Pin_2)
- net VIN: now reaches U1.15 (VIN)
- net VIN: now also J10.1 (Pin_1)
- net SDA: now reaches U1.26 (IO21)
- net SDA: now also J9.4 (Pin_4)
- net SCL: now reaches U1.29 (IO22)
- net SCL: now also J9.3 (Pin_3)
- no-connect marks 18 -> 15
Other:
- note added: "MPU6050"

Commit message: updates
Parts:
- J1: value Conn_01x02_Pin -> flex_01
- J2: value Conn_01x02_Pin -> flex_02
- J3: value Conn_01x02_Pin -> flex_03
- J4: value Conn_01x02_Pin -> flex_04
- J5: value Conn_01x02_Pin -> flex_05
- J6: value Conn_01x02_Pin -> flex_06
- J7: value Conn_01x02_Pin -> flex_07
- J8: value Conn_01x02_Pin -> flex_08
Other:
- note added: "ESP32"
- note added: "Flex Sensors"
- note added: "Power Supply"
- moved on the sheet: J10, J9, U1
